Commit message: fix(URDF): fixed inertia matrix and mass properties

File: source_code/model/Full_Assem.SLDASM/urdf/Full_Assem.SLDASM.urdf (robot description, URDF)
Before this commit: robot Full_Assem.SLDASM, 11 links, 10 joints
Links:
- link base_link: mass 1.2115 -> 1.894
- link link_1: mass 0.356 -> 0.547
- link link_10: mass 0.104537083969092 -> 0.105
- link link_2: mass 0.18671 -> 0.378
- link link_3: mass 0.244673890724835 -> 0.436
- link link_4: mass 0.2446738585482 -> 0.436
- link link_5: mass 0.104537083969092 -> 0.105
- link link_6: mass 0.356003640994798 -> 0.547
- link link_7: mass 0.186708209214479 -> 0.378
- link link_8: mass 0.244673890724774 -> 0.436
- link link_9: mass 0.2446738585482 -> 0.436
