Commit message: feat(Mujoco): added urdf2xml conversion

File: source_code/simulation/model/urdf/Xuanwu.urdf (robot description, URDF)
Before this commit: robot Full_Assem.SLDASM, 11 links, 10 joints
Links:
- link base_link: geometry collision mesh filename=meshes/base_link.STL; visual mesh filename=meshes/base_link.STL
- link link_1: geometry collision mesh filename=meshes/link_1.STL; visual mesh filename=meshes/link_1.STL
- link link_10: geometry collision mesh filename=meshes/link_10.STL; visual mesh filename=meshes/link_10.STL
- link link_2: geometry collision mesh filename=meshes/link_2.STL; visual mesh filename=meshes/link_2.STL
- link link_3: geometry collision mesh filename=meshes/link_3.STL; visual mesh filename=meshes/link_3.STL
- link link_4: geometry collision mesh filename=meshes/link_4.STL; visual mesh filename=meshes/link_4.STL
- link link_5: geometry collision mesh filename=meshes/link_5.STL; visual mesh filename=meshes/link_5.STL
- link link_6: geometry collision mesh filename=meshes/link_6.STL; visual mesh filename=meshes/link_6.STL
- link link_7: geometry collision mesh filename=meshes/link_7.STL; visual mesh filename=meshes/link_7.STL
- link link_8: geometry collision mesh filename=meshes/link_8.STL; visual mesh filename=meshes/link_8.STL
- link link_9: geometry collision mesh filename=meshes/link_9.STL; visual mesh filename=meshes/link_9.STL

Commit message: feat(Mujoco): added XML file and code for urdf2xml

File: source_code/simulation/model/urdf/Xuanwu.urdf (robot description, URDF)
Before this commit: robot Xuanwu, 11 links, 10 joints
Links:
- link base_link: geometry collision mesh filename=./meshes/base_link.STL; visual mesh filename=./meshes/base_link.STL
- link link_1: geometry collision mesh filename=./meshes/link_1.STL; visual mesh filename=./meshes/link_1.STL
- link link_10: geometry collision mesh filename=./meshes/link_10.STL; visual mesh filename=./meshes/link_10.STL
- link link_2: geometry collision mesh filename=./meshes/link_2.STL; visual mesh filename=./meshes/link_2.STL
- link link_3: geometry collision mesh filename=./meshes/link_3.STL; visual mesh filename=./meshes/link_3.STL
- link link_4: geometry collision mesh filename=./meshes/link_4.STL; visual mesh filename=./meshes/link_4.STL
- link link_5: geometry collision mesh filename=./meshes/link_5.STL; visual mesh filename=./meshes/link_5.STL
- link link_6: geometry collision mesh filename=./meshes/link_6.STL; visual mesh filename=./meshes/link_6.STL
- link link_7: geometry collision mesh filename=./meshes/link_7.STL; visual mesh filename=./meshes/link_7.STL
- link link_8: geometry collision mesh filename=./meshes/link_8.STL; visual mesh filename=./meshes/link_8.STL
- link link_9: geometry collision mesh filename=./meshes/link_9.STL; visual mesh filename=./meshes/link_9.STL

Commit message: fix(Mujoco): fixed URDF properties to align with MJCF

File: source_code/simulation/model/urdf/Xuanwu.urdf (robot description, URDF)
Before this commit: robot Xuanwu, 11 links, 10 joints
Links:
- link base_link: geometry collision mesh filename=.../meshes/base_link.STL; visual mesh filename=.../meshes/base_link.STL
- link link_1: geometry collision mesh filename=.../meshes/link_1.STL; visual mesh filename=.../meshes/link_1.STL
- link link_10: geometry collision mesh filename=../meshes/link_10.STL; visual mesh filename=../meshes/link_10.STL
- link link_2: geometry collision mesh filename=../meshes/link_2.STL; visual mesh filename=../meshes/link_2.STL
- link link_3: geometry collision mesh filename=../meshes/link_3.STL; visual mesh filename=../meshes/link_3.STL
- link link_4: geometry collision mesh filename=../meshes/link_4.STL; visual mesh filename=../meshes/link_4.STL
- link link_5: geometry collision mesh filename=../meshes/link_5.STL; visual mesh filename=../meshes/link_5.STL
- link link_6: geometry collision mesh filename=../meshes/link_6.STL; visual mesh filename=../meshes/link_6.STL
- link link_7: geometry collision mesh filename=../meshes/link_7.STL; visual mesh filename=../meshes/link_7.STL
- link link_8: geometry collision mesh filename=../meshes/link_8.STL; visual mesh filename=../meshes/link_8.STL
- link link_9: geometry collision mesh filename=../meshes/link_9.STL; visual mesh filename=../meshes/link_9.STL
Joints:
- joint joint_1: origin xyz=0 0 0 rpy=0 0 0 -> xyz=-0.073 0 -0.001 rpy=0 0 0
- joint joint_10: origin xyz=0 0 0 rpy=0 0 0 -> xyz=0 0 -0.18 rpy=0 0 0
- joint joint_2: origin xyz=0 0 0 rpy=0 0 0 -> xyz=0 -0.083 -0.11 rpy=0 0 0
- joint joint_3: origin xyz=0 0 0 rpy=0 0 0 -> xyz=0 0.082 0 rpy=0 0 0
- joint joint_4: origin xyz=0 0 0 rpy=0 0 0 -> xyz=0 0 -0.18 rpy=0 0 0
- joint joint_5: origin xyz=0 0 0 rpy=0 0 0 -> xyz=0 0 -0.18 rpy=0 0 0
- joint joint_6: origin xyz=0 0 0 rpy=0 0 0 -> xyz=0.073 0 -0.001 rpy=0 0 0
- joint joint_7: origin xyz=0 0 0 rpy=0 0 0 -> xyz=0 -0.083 -0.11 rpy=0 0 0
- joint joint_8: origin xyz=0 0 0 rpy=0 0 0 -> xyz=0 0.082 0 rpy=0 0 0
- joint joint_9: origin xyz=0 0 0 rpy=0 0 0 -> xyz=0 0 -0.18 rpy=0 0 0

Commit message: media(Sim2Sim): updated urdf and mjcf files, added Sim2Sim footage

File: source_code/simulation/model/urdf/Xuanwu.urdf (robot description, URDF)
Before this commit: robot Xuanwu, 11 links, 10 joints
Links:
- link base_link: geometry collision box size=0.1 0.2 0.2; visual mesh filename=../meshes/base_link.STL
- link link_1: geometry visual mesh filename=../meshes/link_1.STL
- link link_2: geometry visual mesh filename=../meshes/link_2.STL
- link link_3: geometry visual mesh filename=../meshes/link_3.STL
- link link_4: geometry visual mesh filename=../meshes/link_4.STL
- link link_6: geometry visual mesh filename=../meshes/link_6.STL
- link link_7: geometry visual mesh filename=../meshes/link_7.STL
- link link_8: geometry visual mesh filename=../meshes/link_8.STL
- link link_9: geometry visual mesh filename=../meshes/link_9.STL

Commit message: feat(URDF): changed some mass properties to align with new 3D printed parts

File: source_code/simulation/model/urdf/Xuanwu.urdf (robot description, URDF)
Before this commit: robot Xuanwu, 11 links, 10 joints
Links:
- link base_link: mass 2.14 -> 1.42
- link link_6: mass 0.574 -> 0.469

Commit message: feat(RL): added new policy

File: source_code/simulation/model/urdf/Xuanwu.urdf (robot description, URDF)
Before this commit: robot Xuanwu, 11 links, 10 joints
Links:
- link link_6: mass 0.469 -> 0.574

Commit message: fix(URDF): corrected mass properties

File: source_code/simulation/model/urdf/Xuanwu.urdf (robot description, URDF)
Before this commit: robot Xuanwu, 11 links, 10 joints
Links:
- link base_link: mass 1.42 -> 1.874
- link link_6: mass 0.574 -> 0.469

Commit message: fix(Models): fixed URDF and MJCF based on true component measurements

File: source_code/simulation/model/urdf/Xuanwu.urdf (robot description, URDF)
Before this commit: robot Xuanwu, 11 links, 10 joints
Links:
- link base_link: mass 1.874 -> 2.016243
- link link_1: mass 0.469 -> 0.504
- link link_10: mass 0.107 -> 0.122
- link link_2: mass 0.364 -> 0.390
- link link_3: mass 0.475 -> 0.481
- link link_4: mass 0.475 -> 0.481
- link link_5: mass 0.107 -> 0.122
- link link_6: mass 0.469 -> 0.504
- link link_7: mass 0.364 -> 0.390
- link link_8: mass 0.475 -> 0.481
- link link_9: mass 0.475 -> 0.481
Joints:
- joint joint_1: origin xyz=-0.073 0 -0.001 rpy=0 0 0 -> xyz=-0.073035 -1.4472E-05 -0.00095242 rpy=0 0 0
- joint joint_10: origin xyz=0 0 -0.18 rpy=0 0 0 -> xyz=-5E-05 1.1901E-05 -0.18002 rpy=0 0 0
- joint joint_2: origin xyz=0 -0.083 -0.11 rpy=0 0 0 -> xyz=4.9294E-05 -0.083183 -0.11003 rpy=0 0 0
- joint joint_3: origin xyz=0 0.082 0 rpy=0 0 0 -> xyz=0.00098795 0.082032 2.035E-05 rpy=0 0 0
- joint joint_4: origin xyz=0 0 -0.18 rpy=0 0 0 -> xyz=5E-05 -5.7742E-05 -0.17996 rpy=0 0 0
- joint joint_5: origin xyz=0 0 -0.18 rpy=0 0 0 -> xyz=5E-05 3.7392E-05 -0.18 rpy=0 0 0
- joint joint_6: origin xyz=0.073 0 -0.001 rpy=0 0 0 -> xyz=0.073035 1.4472E-05 -0.00095242 rpy=0 0 0
- joint joint_7: origin xyz=0 -0.083 -0.11 rpy=0 0 0 -> xyz=-2.035E-05 -0.083212 -0.11003 rpy=0 0 0
- joint joint_8: origin xyz=0 0.082 0 rpy=0 0 0 -> xyz=-0.0010169 0.082032 4.9294E-05 rpy=0 0 0
- joint joint_9: origin xyz=0 0 -0.18 rpy=0 0 0 -> xyz=-5E-05 -1.1901E-05 -0.17998 rpy=0 0 0
